File: usbc-typeshit-1/usbc-typeshit-1.kicad_sch (KiCad schematic)
At the start: 0 parts

Commit message: init pt 2
Parts:
- added U1: IR4302, Package_DFN_QFN:Infineon_PQFN-44-31-5EP_7x7mm_P0.5mm, symbol Amplifier_Audio:IR4302
Connections:
- new net: U1.15 (COM), U1.28 (COM), U1.31 (COM)
- new net: U1.18 (VS1), U1.20 (VS1)
Changed lines of the file:
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@@
 	(generator_version "9.0")
 	(paper "A4")
+	(symbol
+		(lib_id "Amplifier_Audio:IR4302")
+		(at 107.95 83.82 0)
+		(unit 1)
+		(exclude_from_sim no)
+		(in_bom yes)
+		(on_board yes)
+		(dnp no)
+		(fields_autoplaced yes)
+		(property "Reference" "U1"
+			(at 115.1733 60.96 0)
+			(effects
+				(font
+					(size 1.27 1.27)
+				)
+				(justify left)
+			)
+		)
+		(property "Value" "IR4302"
+			(at 115.1733 63.5 0)
+			(effects
+				(font
+					(size 1.27 1.27)
+				)
+				(justify left)
+			)
+		)
+		(property "Footprint" "Package_DFN_QFN:Infineon_PQFN-44-31-5EP_7x7mm_P0.5mm"
+			(at 107.95 83.82 0)
+			(effects
+				(font
+					(size 1.27 1.27)
+					(italic yes)
+				)
+				(hide yes)
+			)
+		)
+		(property "Datasheet" "https://www.infineon.com/dgdl/ir4302.pdf?fileId=5546d462533600a4015355d602a9181d"
+			(at 107.95 83.82 0)
+			(effects
+				(font
+					(size 1.27 1.27)
+				)
+				(hide yes)
+			)
+		)
+		(property "Description" "PowIRaudio 2 Channel Integrated Analog Input Class D Audio Amplifier, 130W/4ohm, 80V, PQFN-44"
+			(at 107.95 83.82 0)
+			(effects
+				(font
+					(size 1.27 1.27)
+				)
+				(hide yes)
+			)
+		)
+		(pin "13"
+		)
+		(pin "21"
+		)
+		(pin "8"
+		)
+		(pin "9"
+		)
+		(pin "30"
+		)
+		(pin "3"
+		)
+		(pin "22"
+		)
+		(pin "5"
+		)
+		(pin "1"
+		)
+		(pin "27"
+		)
+		(pin "26"
+		)
+		(pin "23"
+		)
+		(pin "25"
+		)
+		(pin "28"
+		)
+		(pin "29"
+		)
+		(pin "7"
+		)
+		(pin "31"
+		)
+		(pin "10"
+		)
+		(pin "17"
+		)
+		(pin "18"
+		)
+		(pin "11"
+		)
+		(pin "16"
+		)
+		(pin "15"
+		)
+		(pin "12"
+		)
+		(pin "14"
+		)
+		(pin "2"
+		)
+		(pin "4"
+		)
+		(pin "24"
+		)
+		(pin "20"
+		)
+		(pin "19"
+		)
+		(pin "6"
+		)
+		(instances
+			(project ""
+				(path "/40077179-6726-450b-9792-0bf756987d6f"
+					(reference "U1")
+					(unit 1)
+				)
+			)
+		)
+	)
 	(sheet_instances
 		(path "/"
